File: escpator.kicad_pcb (KiCad board)
At the start: 4 copper layers, 45.7 x 15 mm, 37 parts, among them J1 Conn_01x04_Pin, J2 Conn_02x05_Odd_Even, J3 Conn_01x05, U1 STM32F103CBTx, U4 MCP1700x-330xxTT, Y1 Crystal_GND24

Commit message: aaaaa
Parts:
- moved F1 0.37 mm to (55.0, 39.4)
- moved R27 0.28 mm to (35.9, 41.9)
Routing:
- net /STLINK_TX: track 18.6 -> 12.1 mm
- net +3V3: track 101.3 -> 100.1 mm
- net /LED_STLINK: track 18.8 -> 17.7 mm
- net /STLINK_RX: track 15.0 -> 15.7 mm
- net Earth: track 165.4 -> 165.7 mm, vias 9 -> 10

Commit message: mon28jul1400
Parts:
- C7, C8: moved to B.Cu
- moved C8 3.37 mm to (42.0, 37.0), turned to 0 degrees
- moved C7 2.28 mm to (49.6, 42.8), turned to 180 degrees
- moved R6 1.65 mm to (32.2, 38.9)
- moved C15 1.54 mm to (55.2, 34.3)
- moved R4 1.44 mm to (55.2, 32.8)
- moved R8 0.87 mm to (30.5, 43.0)
- moved R27 0.85 mm to (35.9, 41.0)
- moved R1 0.25 mm to (44.8, 30.9)
- moved C4 0.23 mm to (41.5, 31.9)
- moved R24 0.09 mm to (42.1, 39.5)
Connections:
- J2 pad 9: +5V -> /Pin_navic
- U1 pad 11: unconnected-(U1-PA1-Pad11) -> /Pin_navic
Routing:
- net +5V: track 32.7 -> 7.76 mm, vias 1 -> 0
- net /Pin_navic: track 0.00 -> 19.0 mm, vias 0 -> 2
- net Earth: track 165.7 -> 180.9 mm, vias 10 -> 11
- net /STLINK_RX: track 15.7 -> 13.6 mm
- net Net-(D1-K): track 8.69 -> 7.19 mm
- net /T_JTCK: track 20.7 -> 22.2 mm
- net Net-(J2-Pin_8): track 4.21 -> 5.13 mm

Commit message: b
Parts:
- added R9: 100R, Resistor_SMD:R_0603_1608Metric, B.Cu at (31.0, 41.3)
- R13: moved to B.Cu
- moved R13 2.44 mm to (35.0, 33.5)
- moved C3 2.39 mm to (52.2, 39.1), turned to -135 degrees
- moved R20 2.35 mm to (42.2, 39.5), turned to 0 degrees
- moved R24 1.51 mm to (42.2, 41.0)
Connections:
- J2 pad 9: /Pin_navic -> Net-(J2-Pin_9)
Routing:
- net Net-(J2-Pin_4): track 16.7 -> 8.84 mm, vias 1 -> 0
- net /Pin_navic: track 19.0 -> 14.0 mm, vias 2 -> 1
- net Earth: track 180.9 -> 185.9 mm
- net +3V3: track 100.2 -> 96.6 mm
- net +5V: track 7.76 -> 4.35 mm
- net Net-(J2-Pin_9): track 0.00 -> 3.29 mm, vias 0 -> 1
- net Net-(J2-Pin_7): track 32.3 -> 29.4 mm, vias 2 -> 0
- net /AIN1: track 4.45 -> 5.97 mm
- net /STLINK_TX: track 11.7 -> 12.4 mm
- net /T_JTMS: track 21.0 -> 21.5 mm, vias 2 -> 1

Commit message: c
Parts:
- R9: moved to F.Cu
- moved R13 4.27 mm to (30.8, 33.1)
- moved C10 2.92 mm to (29.9, 36.7), turned to -90 degrees
- moved C5 2.87 mm to (38.9, 33.3)
- moved Y1 2.87 mm to (35.0, 36.8), turned to 0 degrees
- moved R14 2.67 mm to (31.1, 39.7), turned to 90 degrees
- moved C4 2.65 mm to (38.9, 31.8)
- moved C15 2.64 mm to (52.6, 34.3)
- moved R2 2.64 mm to (52.6, 37.2)
- moved R3 2.64 mm to (52.6, 35.7)
- moved R24 2.64 mm to (39.6, 41.0)
- moved C11 2.64 mm to (42.1, 36.3)
- moved C14 2.64 mm to (52.6, 38.7)
- moved C2 2.64 mm to (35.9, 32.4)
- moved C3 2.64 mm to (49.6, 39.2)
- moved C6 2.64 mm to (48.5, 32.1)
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Routing:
- net Earth: track 185.9 -> 149.5 mm, vias 11 -> 9
- net +3V3: track 96.6 -> 78.5 mm, vias 7 -> 8
- net Net-(J2-Pin_2): track 13.1 -> 8.86 mm
- net Net-(J2-Pin_4): track 8.84 -> 4.57 mm
- net Net-(J2-Pin_7): track 29.4 -> 25.3 mm
- net /STLINK_RX: track 13.8 -> 10.4 mm
- net Net-(J1-Pin_1): track 9.97 -> 13.1 mm
- net /Pin_navic: track 14.0 -> 10.9 mm, vias 1 -> 0
- net /OSC_OUT: track 6.93 -> 9.65 mm
- net Net-(J2-Pin_8): track 5.13 -> 2.43 mm
- net /D+: track 10.0 -> 12.6 mm
- net /D-: track 9.75 -> 12.4 mm
- net /AIN1: track 5.97 -> 4.12 mm
- net /OSC_IN?: track 8.90 -> 7.20 mm
- net Net-(J2-Pin_3): track 11.9 -> 10.3 mm
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Other:
- copper layers 4 -> 2

Commit message: d:
Other:
- board text added: "PA1"
- board text removed: "5V"

Commit message: snadfinalverze
Parts:
- moved R24 3.09 mm to (42.6, 40.3), turned to 180 degrees
- moved C3 0.12 mm to (49.5, 39.1)
Routing:
- net /LED_STLINK: track 18.5 -> 17.0 mm, vias 3 -> 1
- net +3V3: track 78.5 -> 77.4 mm

Commit message: e
Parts:
- C10: moved to B.Cu
- moved C10 26.3 mm to (56.1, 34.0), turned to 0 degrees
- moved C3 2.68 mm to (51.9, 37.9), turned to 180 degrees
- moved F1 1.53 mm to (52.2, 41.0)
- moved C1 1.20 mm to (36.1, 40.1), turned to 0 degrees
Routing:
- net Earth: track 149.1 -> 137.2 mm
- net +3V3: track 77.4 -> 80.6 mm, vias 8 -> 7
- net /Pin_navic: track 10.9 -> 9.58 mm
- net +5V: track 4.35 -> 3.65 mm
- net /LED_STLINK: track 17.0 -> 16.3 mm
- net Net-(J1-Pin_1): track 13.1 -> 13.7 mm
