File: escpator.kicad_pcb (KiCad board)
At the start: 2 copper layers, 45.7 x 15 mm, 38 parts, among them J1 Conn_01x04_Pin, J2 Conn_02x05_Odd_Even, J3 Conn_01x05, U1 STM32F103CBTx, U4 MCP1700x-330xxTT, Y1 Crystal_GND24

Commit message: prazdnacommitmessage
Parts:
- C1, C2: value 20pF/6v -> 20pF/50v
- C10, C11, C3, C4, C5, C6, C7, C8: value 100nF/6v -> 100nF/50v
- C14, C15: value 47pF/6v -> 47pF/50v
- C9: value 4.7uF/6v -> 4.7uF/10v
- moved C10 3.81 mm to (52.6, 32.5), turned to 180 degrees
- moved R24 0.10 mm to (42.6, 40.4)
Routing:
- net +3V3: track 80.6 -> 79.8 mm
- net Earth: track 137.1 -> 136.6 mm
