File: escpator.kicad_sch (KiCad schematic)
At the start: 36 parts, among them J1 Conn_01x04_Pin, J2 Conn_02x05_Odd_Even, J3 Conn_01x05, U1 STM32F103CBTx, U3 SRV05-4, U4 MCP1700x-330xxTT, X1 8MHz(12pF)

Commit message: second
Parts:
- removed X1: 8MHz(12pF), Crystal:Crystal_HC49-U_Vertical, symbol Device:Crystal
- added Y1: Crystal_GND24, Crystal:Crystal_SMD_3225-4Pin_3.2x2.5mm_HandSoldering, symbol Device:Crystal_GND24
Connections:
- net Earth: now also Y1.2, Y1.4
- net OSC_IN?: now also Y1.3
- net OSC_OUT: now also Y1.1
Changed lines of the file:
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@@
 	)
 	(junction
+		(at 85.09 55.88)
+		(diameter 0)
+		(color 0 0 0 0)
+	)
+	(junction
 		(at 248.92 33.02)
 		(diameter 0)
@@
 	)
 	(junction
+		(at 90.17 55.88)
+		(diameter 0)
+		(color 0 0 0 0)
+	)
+	(junction
 		(at 201.93 163.83)
 		(diameter 0)
@@
 	(wire
 		(pts
+			(xy 85.09 74.93) (xy 85.09 55.88)
+		)
+		(stroke
+			(width 0)
+			(type default)
+		)
+	)
+	(wire
+		(pts
 			(xy 314.96 86.36) (xy 316.23 86.36)
 		)
@@
 	(wire
 		(pts
+			(xy 85.09 55.88) (xy 90.17 55.88)
+		)
+		(stroke
+			(width 0)
+			(type default)
+		)
+	)
+	(wire
+		(pts
 			(xy 257.81 102.87) (xy 257.81 99.06)
 		)
@@
 	(wire
 		(pts
+			(xy 90.17 55.88) (xy 90.17 64.77)
+		)
+		(stroke
+			(width 0)
+			(type default)
+		)
+	)
+	(wire
+		(pts
 			(xy 236.22 171.45) (xy 270.51 171.45)
 		)
@@
 	(wire
 		(pts
+			(xy 90.17 55.88) (xy 99.06 55.88)
+		)
+		(stroke
+			(width 0)
+			(type default)
+		)
+	)
+	(wire
+		(pts
 			(xy 222.25 21.59) (xy 229.87 21.59)
 		)
@@
 	(wire
 		(pts
+			(xy 90.17 74.93) (xy 85.09 74.93)
+		)
+		(stroke
+			(width 0)
+			(type default)
+		)
+	)
+	(wire
+		(pts
 			(xy 236.22 21.59) (xy 229.87 21.59)
 		)
@@
 	(wire
 		(pts
-			(xy 80.01 55.88) (xy 99.06 55.88)
+			(xy 80.01 55.88) (xy 85.09 55.88)
 		)
 		(stroke
@@
 	)
 	(symbol
+		(lib_id "Device:Crystal_GND24")
+		(at 90.17 69.85 0)
+		(unit 1)
+		(exclude_from_sim no)
+		(in_bom yes)
+		(on_board yes)
+		(dnp no)
+		(fields_autoplaced yes)
+		(property "Reference" "Y1"
+			(at 101.6 63.4298 0)
+			(effects
+				(font
+					(size 1.27 1.27)
+				)
+			)
+		)
+		(property "Value" "Crystal_GND24"
+			(at 101.6 65.9698 0)
+			(effects
+				(font
+					(size 1.27 1.27)
+				)
+			)
+		)
+		(property "Footprint" "Crystal:Crystal_SMD_3225-4Pin_3.2x2.5mm_HandSoldering"
+			(at 90.17 69.85 0)
+			(effects
+				(font
+					(size 1.27 1.27)
+				)
+				(hide yes)
+			)
+		)
+		(property "Datasheet" "~"
+			(at 90.17 69.85 0)
+			(effects
+				(font
+					(size 1.27 1.27)
+				)
+				(hide yes)
+			)
+		)
+		(property "Description" "Four pin crystal, GND on pins 2 and 4"
+			(at 90.17 69.85 0)
+			(effects
+				(font
+					(size 1.27 1.27)
+				)
+				(hide yes)
+			)
+		)
+		(pin "4"
+		)
+		(pin "3"
+		)
+		(pin "1"
+		)
+		(pin "2"
+		)
+		(instances
+			(project ""
+				(path "/7e85dbb0-f9db-48a7-8746-268b4e5d7d4c"
+					(reference "Y1")
+					(unit 1)
+				)
+			)
+		)
+	)
+	(symbol
 		(lib_id "Device:R")
 		(at 229.87 67.31 0)
@@
 					(unit 1)
 				)
-			)
-		)
-	)
-	(symbol
-		(lib_id "Device:Crystal")
-		(at 90.17 69.85 0)
-		(unit 1)
-		(exclude_from_sim no)
-		(in_bom yes)
-		(on_board yes)
-		(dnp no)
-		(property "Reference" "X1"
-			(at 90.17 64.262 0)
-			(effects
-				(font
-					(size 1.27 1.27)
-				)
-			)
-		)
-		(property "Value" "8MHz(12pF)"
-			(at 90.17 66.294 0)
-			(effects
-				(font
-					(size 1.27 1.27)
-				)
-			)
-		)
-		(property "Footprint" "Crystal:Crystal_HC49-U_Vertical"
-			(at 90.17 69.85 0)
-			(effects
-				(font
-					(size 1.27 1.27)
-				)
-				(hide yes)
-			)
-		)
-		(property "Datasheet" "~"
-			(at 90.17 69.85 0)
-			(effects
-				(font
-					(size 1.27 1.27)
-				)
-				(hide yes)
-			)
-		)
-		(property "Description" "Two pin crystal"
-			(at 90.17 69.85 0)
-			(effects
-				(font
-					(size 1.27 1.27)
-				)
-				(hide yes)
-			)
-		)
-		(pin "1"
-		)
-		(pin "2"
-		)
-		(instances
-			(project ""
-				(path "/7e85dbb0-f9db-48a7-8746-268b4e5d7d4c"
-					(reference "X1")
-					(unit 1)
-				)

Commit message: presun LED plus otoceni USB
Connections:
- net D+: now reaches J1.3 (Pin_3), R3.1
- net D-: now reaches J1.2 (Pin_2), R2.1
Changed lines of the file:
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@@
+		)
+	)
+	(label "D+"
+		(at 257.81 99.06 0)
+		(effects
+			(font
+				(size 1.27 1.27)
+			)
+			(justify left bottom)
 		)
 	)
@@
 		(effects
 			(font
+				(size 1.27 1.27)
+			)
+			(justify left bottom)
+		)
+	)
+	(label "D-"
+		(at 256.54 96.52 0)
+		(effects
+			(font

Commit message: changedpins
Parts:
- removed U3: SRV05-4, Package_TO_SOT_SMD:SOT-23-6, symbol Power_Protection:SRV05-4
- added R6, R8: 100R, Resistor_SMD:R_0603_1608Metric, symbol Device:R
Connections:
- net +3V3: now also J2.1 (Pin_1); no longer J2.7 (Pin_7)
- net STLINK_RX: now also R8.1; no longer J2.10 (Pin_10)
- net STLINK_TX: now also R6.1; no longer J2.8 (Pin_8)
- net at R1.1: now also J2.7 (Pin_7); no longer J2.1 (Pin_1)
- new net: J2.10 (Pin_10), R8.2
- new net: J2.8 (Pin_8), R6.2
Other:
- moved on the sheet: R1

Commit message: mon28jul1400
Connections:
- net +5V: no longer J2.9 (Pin_9)
- net Pin_navic: now reaches U1.11 (PA1)
- net Pin_navic: now also J2.9 (Pin_9)
Changed lines of the file:
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@@
+	(wire
+		(pts
+			(xy 172.72 73.66) (xy 190.5 73.66)
+		)
+		(stroke
+			(width 0)
+			(type default)
+		)
+	)
 	(wire
 		(pts
@@
 	(wire
 		(pts
-			(xy 210.82 171.45) (xy 223.52 171.45)
-		)
-		(stroke
-			(width 0)
-			(type default)
-		)
-	)
-	(wire
-		(pts
 			(xy 242.57 33.02) (xy 248.92 33.02)
 		)
@@
 		(pts
 			(xy 300.99 64.77) (xy 304.8 64.77)
+		)
+		(stroke
+			(width 0)
+			(type default)
+		)
+	)
+	(wire
+		(pts
+			(xy 182.88 171.45) (xy 223.52 171.45)
 		)
 		(stroke
@@
 		)
 	)
+	(label "Pin_navic"
+		(at 176.53 73.66 0)
+		(effects
+			(font
+				(size 1.27 1.27)
+			)
+			(justify left bottom)
+		)
+	)
 	(label "T_NRST"
 		(at 177.8 168.91 0)
@@
 	(label "STLINK_TX"
 		(at 176.53 76.2 0)
+		(effects
+			(font
+				(size 1.27 1.27)
+			)
+			(justify left bottom)
+		)
+	)
+	(label "Pin_navic"
+		(at 185.42 171.45 0)
 		(effects
 			(font
@@
 					(unit 1)
 				)
-			)
-		)
-	)
-	(symbol
-		(lib_id "power:+5V")
-		(at 210.82 171.45 90)
-		(unit 1)
-		(exclude_from_sim no)
-		(in_bom yes)
-		(on_board yes)
-		(dnp no)
-		(fields_autoplaced yes)
-		(property "Reference" "#PWR031"
-			(at 214.63 171.45 0)
-			(effects
-				(font
-					(size 1.27 1.27)
-				)
-				(hide yes)
-			)
-		)
-		(property "Value" "+5V"
-			(at 207.01 171.4499 90)
-			(effects
-				(font
-					(size 1.27 1.27)
-				)
-				(justify left)
-			)
-		)
-		(property "Footprint" ""
-			(at 210.82 171.45 0)
-			(effects
-				(font
-					(size 1.27 1.27)
-				)
-				(hide yes)
-			)
-		)
-		(property "Datasheet" ""
-			(at 210.82 171.45 0)
-			(effects
-				(font
-					(size 1.27 1.27)
-				)
-				(hide yes)
-			)
-		)
-		(property "Description" "Power symbol creates a global label with name \"+5V\""
-			(at 210.82 171.45 0)
-			(effects
-				(font
-					(size 1.27 1.27)
-				)
-				(hide yes)
-			)
-		)
-		(pin "1"
-		)
-		(instances
-			(project ""
-				(path "/7e85dbb0-f9db-48a7-8746-268b4e5d7d4c"
-					(reference "#PWR031")
-					(unit 1)
-				)

Commit message: b
Parts:
- added R9: 100R, Resistor_SMD:R_0603_1608Metric, symbol Device:R
Connections:
- net Pin_navic: now also R9.2; no longer J2.9 (Pin_9)
- new net: J2.9 (Pin_9), R9.1
Changed lines of the file:
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@@
 	(wire
 		(pts
+			(xy 213.36 171.45) (xy 223.52 171.45)
+		)
+		(stroke
+			(width 0)
+			(type default)
+		)
+	)
+	(wire
+		(pts
 			(xy 242.57 21.59) (xy 248.92 21.59)
 		)
@@
 	(wire
 		(pts
-			(xy 182.88 171.45) (xy 223.52 171.45)
+			(xy 182.88 171.45) (xy 205.74 171.45)
 		)
 		(stroke
@@
 					(unit 1)
 				)
+			)
+		)
+	)
+	(symbol
+		(lib_id "Device:R")
+		(at 209.55 171.45 270)
+		(unit 1)
+		(exclude_from_sim no)
+		(in_bom yes)
+		(on_board yes)
+		(dnp no)
+		(fields_autoplaced yes)
+		(property "Reference" "R9"
+			(at 209.55 165.1 90)
+			(effects
+				(font
+					(size 1.27 1.27)
+				)
+			)
+		)
+		(property "Value" "100R"
+			(at 209.55 167.64 90)
+			(effects
+				(font
+					(size 1.27 1.27)
+				)
+			)
+		)
+		(property "Footprint" "Resistor_SMD:R_0603_1608Metric"
+			(at 209.55 169.672 90)
+			(effects
+				(font
+					(size 1.27 1.27)
+				)
+				(hide yes)
+			)
+		)
+		(property "Datasheet" "~"
+			(at 209.55 171.45 0)
+			(effects
+				(font
+					(size 1.27 1.27)
+				)
+				(hide yes)
+			)
+		)
+		(property "Description" "Resistor"
+			(at 209.55 171.45 0)
+			(effects
+				(font
+					(size 1.27 1.27)
+				)
+				(hide yes)
+			)
+		)
+		(pin "1"
+		)
+		(pin "2"
+		)
+		(instances
+			(project "escpator"
+				(path "/7e85dbb0-f9db-48a7-8746-268b4e5d7d4c"
+					(reference "R9")
+					(unit 1)
+				)

Commit message: prazdnacommitmessage
Parts:
- C1, C2: value 20pF/6v -> 20pF/50v; LCSC Part # (none) -> C105621
- C10, C11, C3, C4, C5, C6, C7, C8: value 100nF/6v -> 100nF/50v; LCSC Part # (none) -> C14663
- C14, C15: value 47pF/6v -> 47pF/50v; LCSC Part # (none) -> C1671
- C9: value 4.7uF/6v -> 4.7uF/10v; LCSC Part # (none) -> C1705
- D1, D2: LCSC Part # (none) -> C965799
- J1, J2, J3: now left out of the parts list
- R2, R3: LCSC Part # (none) -> C23345
- R26: LCSC Part # (none) -> C22962
- R4: LCSC Part # (none) -> C2906979
- U1: LCSC Part # (none) -> C8304
- Y1: LCSC Part # (none) -> C7275084
Changed lines of the file:
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@@
 			)
 		)
-		(property "Value" "100nF/6v"
+		(property "Value" "100nF/50v"
 			(at 242.824 120.396 0)
 			(effects
@@
 			)
 		)
+		(property "LCSC Part #" "C14663"
+			(at 242.57 115.57 0)
+			(effects
+				(font
+					(size 1.27 1.27)
+				)
+				(hide yes)
+			)
+		)
 		(pin "1"
 		)
@@
 			)
 		)
+		(property "LCSC Part #" "C23345"
+			(at 251.46 102.87 90)
+			(effects
+				(font
+					(size 1.27 1.27)
+				)
+				(hide yes)
+			)
+		)
 		(pin "2"
 		)
@@
 			)
 		)
-		(property "Value" "100nF/6v"
+		(property "Value" "100nF/50v"
 			(at 247.904 38.1 0)
 			(effects
@@
 			)
 		)
+		(property "LCSC Part #" "C14663"
+			(at 248.92 26.67 0)
+			(effects
+				(font
+					(size 1.27 1.27)
+				)
+				(hide yes)
+			)
+		)
 		(pin "2"
 		)
@@
 			)
 		)
+		(property "LCSC Part #" "C965799"
+			(at 297.18 64.77 0)
+			(effects
+				(font
+					(size 1.27 1.27)
+				)
+				(hide yes)
+			)
+		)
 		(pin "2"
 		)
@@
 			)
 		)
-		(property "Value" "20pF/6v"
+		(property "Value" "20pF/50v"
 			(at 83.82 60.9599 0)
 			(effects
@@
 			)
 		)
+		(property "LCSC Part #" "C105621"
+			(at 80.01 59.69 0)
+			(effects
+				(font
+					(size 1.27 1.27)
+				)
+				(hide yes)
+			)
+		)
 		(pin "2"
 		)
@@
 			)
 		)
-		(property "Value" "4.7uF/6v"
+		(property "Value" "4.7uF/10v"
 			(at 219.964 35.052 0)
 			(effects
@@
 			)
 		)
+		(property "LCSC Part #" "C1705"
+			(at 222.25 26.67 0)
+			(effects
+				(font
+					(size 1.27 1.27)
+				)
+				(hide yes)
+			)
+		)
 		(pin "2"
 		)
@@
 		(unit 1)
 		(exclude_from_sim no)
-		(in_bom yes)
+		(in_bom no)
 		(on_board yes)
 		(dnp no)
@@
 			)
 		)
-		(property "Value" "100nF/6v"
+		(property "Value" "100nF/50v"
 			(at 257.81 27.9399 0)
 			(effects
@@
 			)
 		)
+		(property "LCSC Part #" "C14663"
+			(at 254 26.67 0)
+			(effects
+				(font
+					(size 1.27 1.27)
+				)
+				(hide yes)
+			)
+		)
 		(pin "2"
 		)
@@
 		(unit 1)
 		(exclude_from_sim no)
-		(in_bom yes)
+		(in_bom no)
 		(on_board yes)
 		(dnp no)
@@
 			)
 		)
-		(property "Value" "100nF/6v"
+		(property "Value" "100nF/50v"
 			(at 231.902 20.32 0)
 			(effects
@@
 			)
 		)
+		(property "LCSC Part #" "C14663"
+			(at 236.22 26.67 0)
+			(effects
+				(font
+					(size 1.27 1.27)
+				)
+				(hide yes)
+			)
+		)
 		(pin "2"
 		)
@@
 			)
 		)
+		(property "LCSC Part #" "C7275084"
+			(at 90.17 69.85 0)
+			(effects
+				(font
+					(size 1.27 1.27)
+				)
+				(hide yes)
+			)
+		)
 		(pin "4"
 		)
@@
 			)
 		)
-		(property "Value" "100nF/6v"
+		(property "Value" "100nF/50v"
 			(at 121.92 60.9599 0)
 			(effects
@@
 			)
 		)
+		(property "LCSC Part #" "C14663"
+			(at 118.11 59.69 0)
+			(effects
+				(font
+					(size 1.27 1.27)
+				)
+				(hide yes)
+			)
+		)
 		(pin "1"
 		)
@@
 			)
 		)
-		(property "Value" "20pF/6v"
+		(property "Value" "20pF/50v"
 			(at 102.87 60.9599 0)
 			(effects
@@
 			)
 		)
+		(property "LCSC Part #" "C105621"
+			(at 99.06 59.69 0)
+			(effects
+				(font
+					(size 1.27 1.27)
+				)
+				(hide yes)
+			)
+		)
 		(pin "2"
 		)
@@
 			)
 		)
-		(property "Value" "47pF/6v"
+		(property "Value" "47pF/50v"
 			(at 211.582 115.062 0)
 			(effects
@@
 			)
 		)
+		(property "LCSC Part #" "C1671"
+			(at 223.52 115.57 0)
+			(effects
+				(font
+					(size 1.27 1.27)
+				)
+				(hide yes)
+			)
+		)
 		(pin "2"
 		)
@@
 			)
 		)
-		(property "Value" "100nF/6v"
+		(property "Value" "100nF/50v"
 			(at 219.456 19.812 0)
 			(effects
@@
 			)
 		)
+		(property "LCSC Part #" "C14663"
+			(at 229.87 26.67 0)
+			(effects
+				(font
+					(size 1.27 1.27)
+				)
+				(hide yes)
+			)
+		)
 		(pin "2"
 		)
@@
 			)
 		)
-		(property "Value" "100nF/6v"
+		(property "Value" "100nF/50v"
 			(at 242.57 20.066 0)
 			(effects
@@
 			)
 		)
+		(property "LCSC Part #" "C14663"
+			(at 242.57 26.67 0)
+			(effects
+				(font
+					(size 1.27 1.27)
+				)
+				(hide yes)
+			)
+		)
 		(pin "2"
 		)
@@
 			)
 		)
+		(property "LCSC Part #" "C23345"
+			(at 243.84 99.06 90)
+			(effects
+				(font
+					(size 1.27 1.27)
+				)
+				(hide yes)
+			)
+		)
 		(pin "1"
 		)
@@
 			)
 		)
-		(property "Value" "100nF/6v"
+		(property "Value" "100nF/50v"
 			(at 153.67 215.8999 0)
 			(effects
@@
 			)
 		)
+		(property "LCSC Part #" "C14663"
+			(at 149.86 214.63 0)
+			(effects
+				(font
+					(size 1.27 1.27)
+				)
+				(hide yes)
+			)
+		)
 		(pin "1"
 		)
@@
 			)
 		)
+		(property "LCSC Part #" "C8304"
+			(at 154.94 104.14 0)
+			(effects
+				(font
+					(size 1.27 1.27)
+				)
+				(hide yes)
+			)
+		)
 		(pin "1"
 		)
@@
 			)
 		)
+		(property "LCSC Part #" "C22962"
+			(at 120.65 111.76 90)
+			(effects
+				(font
+					(size 1.27 1.27)
+				)
+				(hide yes)
+			)
+		)
 		(pin "2"
 		)
@@
 		(unit 1)
 		(exclude_from_sim no)
-		(in_bom yes)
+		(in_bom no)
 		(on_board yes)
 		(dnp no)
@@
 			)
 		)
+		(property "LCSC Part #" "C965799"
+			(at 297.18 54.61 0)
+			(effects
+				(font
+					(size 1.27 1.27)
+				)
+				(hide yes)
+			)
+		)
 		(pin "1"
 		)
@@
 			)
 		)
+		(property "LCSC Part #" "C2906979"
+			(at 231.14 87.63 0)
+			(effects
+				(font
+					(size 1.27 1.27)
+				)
+				(hide yes)
+			)
+		)
 		(pin "1"
 		)
@@
 			)
 		)
-		(property "Value" "47pF/6v"
+		(property "Value" "47pF/50v"
 			(at 226.314 113.284 0)
 			(effects
@@
 			(at 234.95 115.57 0)
 			(effects
+				(font
+					(size 1.27 1.27)
+				)
+				(hide yes)
+			)
+		)
+		(property "LCSC Part #" "C1671"
+			(at 234.95 115.57 0)
+			(effects
