File: escpator-backups/escpator-2025-07-30_095925/escpator.kicad_pcb (KiCad board)
At the start: 2 copper layers, 45.7 x 15 mm, 38 parts, among them J1 Conn_01x04_Pin, J2 Conn_02x05_Odd_Even, J3 Conn_01x05, U1 STM32F103CBTx, U4 MCP1700x-330xxTT, Y1 Crystal_GND24

Commit message: g
Routing:
- net Net-(D1-K): track 6.74 -> 6.21 mm
Other:
- board text added: "STM_RST"
