File: escpator-backups/escpator-2025-07-30_110642/escpator.kicad_pcb (KiCad board)
At the start: 2 copper layers, 45.7 x 15 mm, 38 parts, among them J1 Conn_01x04_Pin, J2 Conn_02x05_Odd_Even, J3 Conn_01x05, U1 STM32F103CBTx, U4 MCP1700x-330xxTT, Y1 Crystal_GND24

Commit message: g
Other:
- board text added: "STM_RST"
Changed lines of the file:
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@@
 		)
 	)
-	(gr_text "RST"
+	(gr_text "STM_RST"
 		(at 50.5 32.1 90)
 		(layer "B.SilkS")
@@
 	)
 	(segment
-		(start 44.024161 34.674161)
-		(end 43.925314 34.575314)
+		(start 43.4561 34.104686)
+		(end 42.792528 34.104686)
 		(width 0.3)
 		(layer "B.Cu")
@@
 	)
 	(segment
-		(start 40.07776 33.869239)
-		(end 38.647521 32.439)
+		(start 38.259239 32.059239)
+		(end 34.734239 32.059239)
 		(width 0.3)
 		(layer "B.Cu")
@@
 	)
 	(segment
-		(start 45.16 37.56)
-		(end 45.16 36.179338)
+		(start 43.925314 34.575314)
+		(end 43.925314 34.5739)
 		(width 0.3)
 		(layer "B.Cu")
@@
 	)
 	(segment
-		(start 44.024161 35.043499)
-		(end 44.024161 34.674161)
+		(start 42.792528 34.104686)
+		(end 42.557081 33.869239)
 		(width 0.3)
 		(layer "B.Cu")
@@
 	)
 	(segment
-		(start 33.693478 33.1)
-		(end 31.625 33.1)
+		(start 42.557081 33.869239)
+		(end 40.07776 33.869239)
 		(width 0.3)
 		(layer "B.Cu")
@@
 	)
 	(segment
-		(start 46.84 38.39)
-		(end 45.99 38.39)
+		(start 45.16 36.179338)
+		(end 44.024161 35.043499)
 		(width 0.3)
 		(layer "B.Cu")
@@
 	)
 	(segment
-		(start 38.259239 32.059239)
-		(end 34.734239 32.059239)
+		(start 45.16 36.46)
+		(end 45.16 36.179338)
 		(width 0.3)
 		(layer "B.Cu")
@@
 	)
 	(segment
-		(start 45.16 36.179338)
-		(end 44.024161 35.043499)
+		(start 38.639 32.439)
+		(end 38.259239 32.059239)
 		(width 0.3)
 		(layer "B.Cu")
@@
 	)
 	(segment
-		(start 34.734239 32.059239)
-		(end 33.693478 33.1)
+		(start 44.024161 34.674161)
+		(end 43.925314 34.575314)
 		(width 0.3)
 		(layer "B.Cu")
@@
 	)
 	(segment
-		(start 43.925314 34.5739)
-		(end 43.220653 33.869239)
+		(start 38.647521 32.439)
+		(end 38.639 32.439)
 		(width 0.3)
 		(layer "B.Cu")
@@
 	)
 	(segment
-		(start 43.220653 33.869239)
-		(end 40.07776 33.869239)
+		(start 46.84 38.39)
+		(end 46.84 38.14)
 		(width 0.3)
 		(layer "B.Cu")
@@
 	)
 	(segment
-		(start 43.925314 34.575314)
-		(end 43.925314 34.5739)
+		(start 33.693478 33.1)
+		(end 31.625 33.1)
 		(width 0.3)
 		(layer "B.Cu")
@@
 	)
 	(segment
-		(start 38.647521 32.439)
-		(end 38.639 32.439)
+		(start 43.925314 34.5739)
+		(end 43.4561 34.104686)
 		(width 0.3)
 		(layer "B.Cu")
@@
 	)
 	(segment
-		(start 38.639 32.439)
-		(end 38.259239 32.059239)
+		(start 40.07776 33.869239)
+		(end 38.647521 32.439)
 		(width 0.3)
 		(layer "B.Cu")
@@
 	)
 	(segment
-		(start 45.99 38.39)
-		(end 45.16 37.56)
+		(start 34.734239 32.059239)
+		(end 33.693478 33.1)
+		(width 0.3)
+		(layer "B.Cu")
+		(net 19)
+	)
+	(segment
+		(start 46.84 38.14)
+		(end 45.16 36.46)
+		(width 0.3)
+		(layer "B.Cu")
+		(net 19)
+	)
+	(segment
+		(start 44.024161 35.043499)
+		(end 44.024161 34.674161)
 		(width 0.3)
 		(layer "B.Cu")
@@
 	)
 	(segment
-		(start 44.784669 39.834669)
-		(end 44.429239 39.479239)
+		(start 38.44 32.94)
+		(end 37.415 32.94)
 		(width 0.3)
 		(layer "B.Cu")
@@
 	)
 	(segment
-		(start 42.620239 34.370239)
-		(end 39.87024 34.370239)
+		(start 44.784669 39.834669)
+		(end 44.429239 39.479239)
 		(width 0.3)
 		(layer "B.Cu")
@@
 	)
 	(segment
+		(start 39.87024 34.370239)
+		(end 38.44 32.94)
+		(width 0.3)
+		(layer "B.Cu")
+		(net 22)
+	)
+	(segment
 		(start 44.784669 39.909239)
 		(end 44.784669 39.834669)
@@
 	)
 	(segment
-		(start 39.87024 34.370239)
-		(end 38.44 32.94)
+		(start 42.855686 34.605686)
+		(end 42.585008 34.605686)
 		(width 0.3)
 		(layer "B.Cu")
@@
 	)
 	(segment
-		(start 38.44 32.94)
-		(end 37.415 32.94)
+		(start 42.585008 34.605686)
+		(end 42.34956 34.370239)
 		(width 0.3)
 		(layer "B.Cu")
@@
 	)
 	(segment
+		(start 42.34956 34.370239)
+		(end 39.87024 34.370239)
+		(width 0.3)
+		(layer "B.Cu")
+		(net 22)
+	)
+	(segment
 		(start 43.124314 34.874314)
-		(end 42.620239 34.370239)
+		(end 42.855686 34.605686)
 		(width 0.3)
 		(layer "B.Cu")
@@
 		(layers "F.Cu" "B.Cu")
 		(hatch edge 0.5)
-		(connect_pads yes
-			(clearance 0.254)
+		(connect_pads
+			(clearance 0.508)
 		)
 		(min_thickness 0.25)
@@
 		(polygon
 			(pts
-				(xy 52.330761 29.630761) (xy 54.530761 29.630761) (xy 54.530761 31.040761) (xy 58.630761 31.030761)
-				(xy 58.630761 43.230761) (xy 54.530761 43.230761) (xy 54.530761 44.630761) (xy 32.05 44.630761)
-				(xy 24.430761 44.630761) (xy 24.430761 29.630761)
+				(xy 46.730761 29.630761) (xy 46.680761 32.430761) (xy 50.670761 32.430761) (xy 50.670761 31.160761)
+				(xy 52.330761 31.130761) (xy 52.330761 29.630761) (xy 54.530761 29.630761) (xy 54.530761 31.040761)
+				(xy 58.630761 31.030761) (xy 58.630761 32.730761) (xy 58.6 35.03) (xy 58.630761 43.230761) (xy 54.530761 43.230761)
+				(xy 54.530761 44.630761) (xy 32.05 44.630761) (xy 29.85 44.65) (xy 24.430761 44.630761) (xy 24.430761 29.630761)
 			)
 		)
