File: escpator-backups/escpator-2025-07-30_121541/escpator.kicad_pcb (KiCad board)
At the start: 2 copper layers, 45.7 x 15 mm, 38 parts, among them J1 Conn_01x04_Pin, J2 Conn_02x05_Odd_Even, J3 Conn_01x05, U1 STM32F103CBTx, U4 MCP1700x-330xxTT, Y1 Crystal_GND24

Commit message: g
Parts:
- added REF**: Tab, PCM_kikit:Tab, F.Cu at (30.5, 46.4)
- added REF**: Tab, PCM_kikit:Tab, F.Cu at (30.0, 29.7)
- added REF**: Tab, PCM_kikit:Tab, F.Cu at (50.0, 29.6)
- added REF**: Tab, PCM_kikit:Tab, F.Cu at (30.0, 44.7)
Other:
- board text added: "STM_RST"
